File: system_development/Charleston/V0.1/V0.1/Battery Testing-BMS system V.01/Battery Testing-BMS system V.01.kicad_pcb (KiCad board)
At the start: 2 copper layers, 34.8 x 64.4 mm, 6 parts, among them J1 Screw_Terminal_01x12

Commit message: Fixed
Fixed issues with board
Parts:
- removed REF** (x2): MountingHole_2.5mm, MountingHole:MountingHole_2.5mm
- moved G*** 0.65 mm to (123.8, 123.6)
Connections:
- J1 pad 1: Net-(J1-Pin_1) -> GND
- J1 pad 7: GND -> Net-(J1-Pin_7)
- U1 pad 1: Net-(J1-Pin_1) -> GND
- U1 pad 7: GND -> Net-(J1-Pin_7)
Routing:
- net Net-(J1-Pin_1): track 23.5 -> 0.00 mm
- net Net-(J1-Pin_11): track 23.9 -> 47.1 mm
- net Net-(J1-Pin_10): track 23.3 -> 0.00 mm
- net Net-(J1-Pin_7): track 0.00 -> 21.5 mm
- net Net-(J1-Pin_6): track 20.9 -> 42.0 mm
- net Net-(J1-Pin_5): track 21.1 -> 0.00 mm
- removed copper zone on F.Cu, net GND
Other:
- board size 34.8 x 64.4 mm -> 36.1 x 64.4 mm

Commit message: trying
Routing:
- net Net-(J1-Pin_11): track 47.1 -> 23.9 mm
- net Net-(J1-Pin_10): track 0.00 -> 23.3 mm
- net Net-(J1-Pin_6): track 42.0 -> 20.9 mm
- net Net-(J1-Pin_5): track 0.00 -> 21.1 mm
Changed lines of the file:
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@@
   (net 9 "Net-(J1-Pin_11)")
   (net 10 "GND")
+  (net 11 "Net-(J1-Pin_5)")
+  (net 12 "Net-(J1-Pin_10)")
   (footprint "BMS_PCB_Library:Altech_AK300_1x12_P5.00mm_45-Degree" (layer "F.Cu")
     (at 136.767 66.357 -90)
@@
       (net 5 "Net-(J1-Pin_4)") (pinfunction "Pin_4") (pintype "passive"))
     (pad "5" thru_hole circle (at 20 0 270) (size 3 3) (drill 1.5) (layers "*.Cu" "*.Mask")
-      (net 4 "Net-(J1-Pin_5)") (pinfunction "Pin_5") (pintype "passive"))
+      (net 11 "Net-(J1-Pin_5)") (pinfunction "Pin_5") (pintype "passive"))
     (pad "6" thru_hole circle (at 25 0 270) (size 3 3) (drill 1.5) (layers "*.Cu" "*.Mask")
       (net 4 "Net-(J1-Pin_6)") (pinfunction "Pin_6") (pintype "passive"))
@@
       (net 1 "Net-(J1-Pin_9)") (pinfunction "Pin_9") (pintype "passive"))
     (pad "10" thru_hole circle (at 45 0 270) (size 3 3) (drill 1.5) (layers "*.Cu" "*.Mask")
-      (net 9 "Net-(J1-Pin_10)") (pinfunction "Pin_10") (pintype "passive"))
+      (net 12 "Net-(J1-Pin_10)") (pinfunction "Pin_10") (pintype "passive"))
     (pad "11" thru_hole circle (at 50 0 270) (size 3 3) (drill 1.5) (layers "*.Cu" "*.Mask")
       (net 9 "Net-(J1-Pin_11)") (pinfunction "Pin_11") (pintype "passive"))
@@
       (net 5 "Net-(J1-Pin_4)") (pintype "input"))
     (pad "5" smd rect (at -5.334 5.588 270) (size 1.5 10) (layers "F.Cu" "F.Paste" "F.Mask")
-      (net 4 "Net-(J1-Pin_5)") (pintype "input"))
+      (net 11 "Net-(J1-Pin_5)") (pintype "input"))
     (pad "6" smd rect (at -1.778 5.588 270) (size 1.5 10) (layers "F.Cu" "F.Paste" "F.Mask")
       (net 4 "Net-(J1-Pin_6)") (pintype "input"))
@@
       (net 1 "Net-(J1-Pin_9)") (pintype "input"))
     (pad "10" smd rect (at 12.446 5.588 270) (size 1.5 10) (layers "F.Cu" "F.Paste" "F.Mask")
-      (net 9 "Net-(J1-Pin_10)") (pintype "input"))
+      (net 12 "Net-(J1-Pin_10)") (pintype "input"))
     (pad "11" smd rect (at 16.002 5.588 270) (size 1.5 10) (layers "F.Cu" "F.Paste" "F.Mask")
       (net 9 "Net-(J1-Pin_11)") (pintype "input"))
@@
   (segment (start 116.078 90.932) (end 136.342 90.932) (width 0.25) (layer "F.Cu") (net 4))
   (segment (start 136.342 90.932) (end 136.767 91.357) (width 0.25) (layer "F.Cu") (net 4))
-  (segment (start 116.078 87.376) (end 135.748 87.376) (width 0.25) (layer "F.Cu") (net 4))
-  (segment (start 135.748 87.376) (end 136.767 86.357) (width 0.25) (layer "F.Cu") (net 4))
   (segment (start 116.078 83.82) (end 134.304 83.82) (width 0.25) (layer "F.Cu") (net 5))
   (segment (start 134.304 83.82) (end 136.767 81.357) (width 0.25) (layer "F.Cu") (net 5))
@@
   (segment (start 116.078 108.712) (end 129.122 108.712) (width 0.25) (layer "F.Cu") (net 9))
   (segment (start 129.122 108.712) (end 136.767 116.357) (width 0.25) (layer "F.Cu") (net 9))
-  (segment (start 116.078 105.156) (end 130.566 105.156) (width 0.25) (layer "F.Cu") (net 9))
-  (segment (start 130.566 105.156) (end 136.767 111.357) (width 0.25) (layer "F.Cu") (net 9))
+  (segment (start 116.078 87.376) (end 135.748 87.376) (width 0.25) (layer "F.Cu") (net 11))
+  (segment (start 135.748 87.376) (end 136.767 86.357) (width 0.25) (layer "F.Cu") (net 11))
+  (segment (start 116.078 105.156) (end 130.566 105.156) (width 0.25) (layer "F.Cu") (net 12))
+  (segment (start 130.566 105.156) (end 136.767 111.357) (width 0.25) (layer "F.Cu") (net 12))
 )
